File: LoRa_Transceiver.sch (KiCad schematic (older format))
At the start: 0 parts

Commit message: Fix atmo sensor, add LoRa schematic
Parts:
- added C?: C, symbol Device:C
- added C? (x3): 100n, symbol Device:C
- added L?: L, symbol Device:L
- added R?: 10K, symbol Device:R
- added U?: SX1262, symbol co2_sensor_node:SX1262
- added Y?: Q22FA1280001800, symbol Device:Crystal_GND2
Connections:
- new net: R?.2, U?.15 (nRESET)
- new net: U?.3 (XTA), Y?.1
- new net: U?.4 (XTB), Y?.3
- new net: C?.1, L?.1, U?.7 (VREG)
- new net: L?.2, U?.9 (DCC_SW)
- new net +3V3: C?.1, C?.1, C?.1, R?.1, U?.1 (VDD_IN), U?.10 (VBAT), U?.11 (VBAT_IO)
- new net BUSY: U?.14 (BUSY)
- new net CSN: U?.19 (nCS)
- new net DIO2: U?.12 (DIO2)
- new net GND: C?.2, C?.2, C?.2, C?.2, U?.2 (GND), U?.20 (GND), U?.25 (GND_PAD), U?.5 (GND), U?.8 (GND), Y?.2
- new net IRQ1: U?.13 (DIO1)
- new net IRQ2: U?.6 (DIO3)
- new net MISO: U?.16 (MISO)
- new net MOSI: U?.17 (MOSI)
- new net SCLK: U?.18 (SCK)
