File: SD_card.sch (KiCad schematic (older format))
At the start: 0 parts

Commit message: Rearranged IO connections to take advantage of hardware interfaces where possible
Parts:
- added J?: TF-15x15, symbol Connector:Micro_SD_Card_Det
Changed lines of the file:
@@
 Comment4 ""
 $EndDescr
+$Comp
+L Connector:Micro_SD_Card_Det J?
+U 1 1 60B61966
+P 7900 4000
+F 0 "J?" H 7850 4817 50  0000 C CNN
+F 1 "TF-15x15" H 7850 4726 50  0000 C CNN
+F 2 "" H 9950 4700 50  0001 C CNN
+F 3 "https://datasheet.lcsc.com/szlcsc/2009111836_SOFNG-TF-15x15_C111196.pdf" H 7900 4100 50  0001 C CNN
+F 4 "https://lcsc.com/product-detail/Card-Sockets-Connectors_SOFNG-TF-15x15_C111196.html/?href=jlc-SMT" H 7900 4000 50  0001 C CNN "LCSC"
+	1    7900 4000
+	1    0    0    -1
+$EndComp
 $EndSCHEMATC
