File: Status_LED.kicad_sch (KiCad schematic)
At the start: 2 parts

Commit message: Add testpoint footprint assignments
Parts:
- gave numbers to parts that had none: 2
Changed lines of the file:
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@@
   (symbol (lib_id "Device:R") (at 111.76 90.17 270) (unit 1)
     (in_bom yes) (on_board yes) (fields_autoplaced)
-    (property "Reference" "R?" (id 0) (at 111.76 85.4542 90))
+    (property "Reference" "R16" (id 0) (at 111.76 85.4542 90))
     (property "Value" "1k" (id 1) (at 111.76 87.9911 90))
     (property "Footprint" "Resistor_SMD:R_0603_1608Metric" (id 2) (at 111.76 88.392 90)
@@
   (symbol (lib_id "power:GND") (at 132.08 93.98 0) (unit 1)
     (in_bom yes) (on_board yes) (fields_autoplaced)
-    (property "Reference" "#PWR?" (id 0) (at 132.08 100.33 0)
+    (property "Reference" "#PWR0126" (id 0) (at 132.08 100.33 0)
       (effects (font (size 1.27 1.27)) hide)
     )
@@
   (symbol (lib_id "Device:LED") (at 124.46 90.17 180) (unit 1)
     (in_bom yes) (on_board yes) (fields_autoplaced)
-    (property "Reference" "D?" (id 0) (at 126.0475 84.3112 0))
+    (property "Reference" "D1" (id 0) (at 126.0475 84.3112 0))
     (property "Value" "Green LED" (id 1) (at 126.0475 86.8481 0))
     (property "Footprint" "LED_SMD:LED_0603_1608Metric" (id 2) (at 124.46 90.17 0)

Commit message: Finalize schematic
Other:
- title: (none) -> CO2 Chamber - Status LED
Changed lines of the file:
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@@
 (kicad_sch (version 20211123) (generator eeschema)
   (paper "A4")
+  (title_block
+    (title "CO2 Chamber - Status LED")
+    (date "2022-05-20")
+    (rev "1")
+  )
   (wire (pts (xy 115.57 90.17) (xy 120.65 90.17))
     (stroke (width 0) (type default) (color 0 0 0 0))
